File: pcb/HP203B-I2C-sensor.kicad_sch (KiCad schematic)
At the start: 7 parts, among them J1 Conn_01x04_Socket, J2 Conn_01x04_Pin, J3 Conn_01x04_Socket

Commit message: polish a bit
Parts:
- C1: value 4.1u -> 4.7u
Changed lines of the file:
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@@
 			)
 		)
-		(property "Value" "4.1u"
+		(property "Value" "4.7u"
 			(at 144.78 78.74 90)
 			(show_name no)
